File: HW3/433_PIC/NEWNU32.sch (EAGLE design)
At the start: 0 parts

Commit message: Starting work on creating a New NU32 PCB for HW2
Populated Library, created a schematic, and started a board file in Eagle
Parts:
- added C1, C2: 0.1 uF, 433:C-US025-025X050
- added C3, C4: 0.1uF, 433:C-US025-025X050
- added C5, C6: 10uF, 433:CPOL-USB45181B
- added J1: USB-MB-H, 433:USB-MB-H
- added LED1: Red, led:LED3MM
- added LED2: Green, led:LED3MM
- added R1, R2: 10k, 433:R-US_0207/10
- added R3, R4: 330, 433:R-US_0207/10
- added U$1: PIC32MX250F128B, 433:PIC32MX250F128B
- added U$2: SLIDE, 433:SLIDE
- added U$3: MCP1702, 433:MCP1702
- added U$4: USER, 433:PB
- added U$5: RESET, 433:PB
- added U$6, U$7: CONN_08, 433:CONN_08
- added U$8: PICKIT3, 433:PICKIT3
- added U$9: 8MHz, 433:OSC
Connections:
- new net +3V3: C1.1, C2.1, C4.1, C6.+, LED1.A, R1.2, R2.2, U$1.13.VDD, U$1.23.VUSB3V3, U$1.28.AVDD, U$3.3.VOUT, U$7.2, U$8.VDD
- new net +5V: C3.1, U$1.15.VBUS, U$2.3, U$3.2.VIN, U$6.2
- new net A0: U$1.2.A0, U$7.8
- new net A1: U$1.3.A1, U$7.7
- new net A4/LED: LED2.A, U$1.12.A4/LED
- new net A4/USER: U$7.3
- new net B13: U$1.24.B13, U$6.6
- new net B14: U$1.25.B14, U$6.7
- new net B15: U$1.26.B15, U$6.8
- new net B2: U$1.6.B2, U$7.6
- new net B3: U$1.7.B3, U$7.5
- new net B4/USER: R1.1, U$1.11.B4/USER, U$4.1, U$7.4
- new net B7: U$1.16.B7, U$6.3
- new net B8: U$1.17.B8, U$6.4
- new net B9: U$1.18.B9, U$6.5
- new net D+: J1.D+, U$1.21.D+/B10
- new net D-: J1.D-, U$1.D-/B11
- new net GND: C1.2, C2.2, C3.2, C4.2, C5.-, C6.-, J1.GND, R3.2, R4.2, U$1.19.VSS, U$1.27.AVSS, U$1.8.VSS, U$3.1.GND, U$4.2, U$5.2, U$6.1, U$7.1, U$8.GND, U$9.2.GND
- new net MCLR: R2.1, U$1.1.MCLR, U$5.1, U$8.MCLR
- new net N$1: LED2.C, R4.1
- new net N$2: LED1.C, R3.1
- new net N$3: U$1.9.OSC1/A2, U$9.1.OSC1
- new net N$4: U$1.10.OSC2/A3, U$9.3.OSC2
- new net N$6: C5.+, U$1.20.VCAP
- new net PGC: U$1.5.PGC/B1, U$8.PGC
- new net PGD: U$1.4.PGD/B0, U$8.PGD
- new net USBID: J1.ID, U$1.14.USBID/B6
- new net VB: J1.VBUS, U$2.2
