File: HW3/433_PIC/NEWNU32.sch (EAGLE design)
At the start: 22 parts, among them J1 USB-MB-H

Commit message: Finished Initial Board
Connections:
- removed net A4/USER: U$7.3
- net A4/LED: now also U$7.3
- net D-: now also U$1.22.D-/B11; no longer U$1.D-/B11
Other:
- moved on the sheet: C2, U$7
Changed lines of the file:
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@@
 <instance part="R4" gate="G$1" x="259.08" y="15.24" rot="R90"/>
 <instance part="C1" gate="G$1" x="15.24" y="15.24"/>
-<instance part="C2" gate="G$1" x="86.36" y="76.2"/>
+<instance part="C2" gate="G$1" x="83.82" y="76.2"/>
 <instance part="C3" gate="G$1" x="147.32" y="-10.16" rot="MR0"/>
 <instance part="C4" gate="G$1" x="198.12" y="-10.16" rot="MR0"/>
@@
 <instance part="C6" gate="G$1" x="205.74" y="-10.16" rot="MR0"/>
 <instance part="U$6" gate="G$1" x="144.78" y="71.12"/>
-<instance part="U$7" gate="G$1" x="144.78" y="38.1"/>
+<instance part="U$7" gate="G$1" x="127" y="71.12" rot="MR0"/>
 <instance part="U$8" gate="G$1" x="-10.16" y="68.58"/>
 <instance part="U$9" gate="G$1" x="-15.24" y="30.48"/>
@@
 <instance part="GND16" gate="1" x="220.98" y="40.64"/>
 <instance part="GND17" gate="1" x="220.98" y="71.12"/>
-<instance part="GND18" gate="1" x="152.4" y="27.94"/>
+<instance part="GND18" gate="1" x="119.38" y="60.96" rot="MR0"/>
 <instance part="GND19" gate="1" x="154.94" y="60.96"/>
 <instance part="P+1" gate="1" x="129.54" y="2.54" rot="MR0"/>
@@
 <instance part="+3V5" gate="G$1" x="185.42" y="66.04"/>
 <instance part="+3V6" gate="G$1" x="185.42" y="101.6"/>
-<instance part="+3V7" gate="G$1" x="157.48" y="35.56"/>
+<instance part="+3V7" gate="G$1" x="114.3" y="68.58" rot="MR0"/>
 <instance part="P+3" gate="1" x="162.56" y="68.58"/>
 <instance part="+3V8" gate="G$1" x="91.44" y="55.88"/>
@@
 <pinref part="C2" gate="G$1" pin="2"/>
 <pinref part="GND8" gate="1" pin="GND"/>
-<wire x1="86.36" y1="71.12" x2="88.9" y2="71.12" width="0.1524" layer="91"/>
+<wire x1="83.82" y1="71.12" x2="88.9" y2="71.12" width="0.1524" layer="91"/>
 </segment>
 <segment>
@@
 <pinref part="U$7" gate="G$1" pin="1"/>
 <pinref part="GND18" gate="1" pin="GND"/>
-<wire x1="149.86" y1="30.48" x2="152.4" y2="30.48" width="0.1524" layer="91"/>
+<wire x1="121.92" y1="63.5" x2="119.38" y2="63.5" width="0.1524" layer="91"/>
 </segment>
 <segment>
@@
 </segment>
 <segment>
+<pinref part="U$8" gate="G$1" pin="VDD"/>
+<pinref part="+3V3" gate="G$1" pin="+3V3"/>
+<wire x1="-10.16" y1="73.66" x2="-17.78" y2="73.66" width="0.1524" layer="91"/>
+</segment>
+<segment>
+<pinref part="R2" gate="G$1" pin="2"/>
+<pinref part="+3V6" gate="G$1" pin="+3V3"/>
+<wire x1="185.42" y1="93.98" x2="185.42" y2="99.06" width="0.1524" layer="91"/>
+</segment>
+<segment>
+<pinref part="+3V5" gate="G$1" pin="+3V3"/>
+<pinref part="R1" gate="G$1" pin="2"/>
+<wire x1="185.42" y1="63.5" x2="185.42" y2="60.96" width="0.1524" layer="91"/>
+</segment>
+<segment>
+<pinref part="U$7" gate="G$1" pin="2"/>
+<pinref part="+3V7" gate="G$1" pin="+3V3"/>
+<wire x1="121.92" y1="66.04" x2="114.3" y2="66.04" width="0.1524" layer="91"/>
+</segment>
+<segment>
 <pinref part="U$1" gate="G$1" pin="28.AVDD"/>
 <pinref part="C2" gate="G$1" pin="1"/>
-<wire x1="68.58" y1="78.74" x2="86.36" y2="78.74" width="0.1524" layer="91"/>
+<wire x1="68.58" y1="78.74" x2="83.82" y2="78.74" width="0.1524" layer="91"/>
 <pinref part="+3V2" gate="G$1" pin="+3V3"/>
-<wire x1="86.36" y1="78.74" x2="91.44" y2="78.74" width="0.1524" layer="91"/>
+<wire x1="83.82" y1="78.74" x2="91.44" y2="78.74" width="0.1524" layer="91"/>
 <wire x1="91.44" y1="78.74" x2="91.44" y2="81.28" width="0.1524" layer="91"/>
-<junction x="86.36" y="78.74"/>
+<junction x="83.82" y="78.74"/>
 </segment>
 <segment>
@@
 <pinref part="+3V8" gate="G$1" pin="+3V3"/>
 <wire x1="68.58" y1="53.34" x2="91.44" y2="53.34" width="0.1524" layer="91"/>
-</segment>
-<segment>
-<pinref part="U$8" gate="G$1" pin="VDD"/>
-<pinref part="+3V3" gate="G$1" pin="+3V3"/>
-<wire x1="-10.16" y1="73.66" x2="-17.78" y2="73.66" width="0.1524" layer="91"/>
-</segment>
-<segment>
-<pinref part="R2" gate="G$1" pin="2"/>
-<pinref part="+3V6" gate="G$1" pin="+3V3"/>
-<wire x1="185.42" y1="93.98" x2="185.42" y2="99.06" width="0.1524" layer="91"/>
-</segment>
-<segment>
-<pinref part="+3V5" gate="G$1" pin="+3V3"/>
-<pinref part="R1" gate="G$1" pin="2"/>
-<wire x1="185.42" y1="63.5" x2="185.42" y2="60.96" width="0.1524" layer="91"/>
-</segment>
-<segment>
-<pinref part="U$7" gate="G$1" pin="2"/>
-<pinref part="+3V7" gate="G$1" pin="+3V3"/>
-<wire x1="149.86" y1="33.02" x2="157.48" y2="33.02" width="0.1524" layer="91"/>
 </segment>
 </net>
@@
 <segment>
 <pinref part="U$7" gate="G$1" pin="8"/>
-<wire x1="149.86" y1="48.26" x2="160.02" y2="48.26" width="0.1524" layer="91"/>
-<label x="157.48" y="48.26" size="1.778" layer="95"/>
+<wire x1="121.92" y1="81.28" x2="111.76" y2="81.28" width="0.1524" layer="91"/>
+<label x="114.3" y="81.28" size="1.778" layer="95" rot="MR0"/>
 </segment>
 </net>
@@
 <segment>
 <pinref part="U$7" gate="G$1" pin="7"/>
-<wire x1="149.86" y1="45.72" x2="160.02" y2="45.72" width="0.1524" layer="91"/>
-<label x="157.48" y="45.72" size="1.778" layer="95"/>
+<wire x1="121.92" y1="78.74" x2="111.76" y2="78.74" width="0.1524" layer="91"/>
+<label x="114.3" y="78.74" size="1.778" layer="95" rot="MR0"/>
 </segment>
 </net>
@@
 <segment>
 <pinref part="U$7" gate="G$1" pin="6"/>
-<wire x1="149.86" y1="43.18" x2="160.02" y2="43.18" width="0.1524" layer="91"/>
-<label x="157.48" y="43.18" size="1.778" layer="95"/>
+<wire x1="121.92" y1="76.2" x2="111.76" y2="76.2" width="0.1524" layer="91"/>
+<label x="114.3" y="76.2" size="1.778" layer="95" rot="MR0"/>
 </segment>
 </net>
@@
 <segment>
 <pinref part="U$7" gate="G$1" pin="5"/>
-<wire x1="149.86" y1="40.64" x2="160.02" y2="40.64" width="0.1524" layer="91"/>
-<label x="157.48" y="40.64" size="1.778" layer="95"/>
+<wire x1="121.92" y1="73.66" x2="111.76" y2="73.66" width="0.1524" layer="91"/>
+<label x="114.3" y="73.66" size="1.778" layer="95" rot="MR0"/>
 </segment>
 </net>
@@
 <segment>
 <pinref part="U$7" gate="G$1" pin="4"/>
-<wire x1="149.86" y1="38.1" x2="160.02" y2="38.1" width="0.1524" layer="91"/>
-<label x="157.48" y="38.1" size="1.778" layer="95"/>
+<wire x1="121.92" y1="71.12" x2="111.76" y2="71.12" width="0.1524" layer="91"/>
+<label x="114.3" y="71.12" size="1.778" layer="95" rot="MR0"/>
 </segment>
 </net>
@@
 <label x="261.62" y="-10.16" size="1.778" layer="95"/>
 </segment>
+<segment>
+<pinref part="U$7" gate="G$1" pin="3"/>
+<wire x1="121.92" y1="68.58" x2="119.38" y2="68.58" width="0.1524" layer="91"/>
+<label x="121.92" y="68.58" size="1.778" layer="95" rot="MR0"/>
+</segment>
 </net>
 <net name="USBID" class="0">
@@
 <net name="D-" class="0">
 <segment>
-<pinref part="U$1" gate="G$1" pin="D-/B11"/>
+<pinref part="U$1" gate="G$1" pin="22.D-/B11"/>
 <wire x1="68.58" y1="48.26" x2="78.74" y2="48.26" width="0.1524" layer="91"/>
 <label x="78.74" y="48.26" size="1.778" layer="95"/>
@@
 </segment>
 </net>
-<net name="A4/USER" class="0">
-<segment>
-<pinref part="U$7" gate="G$1" pin="3"/>
-<wire x1="149.86" y1="35.56" x2="152.4" y2="35.56" width="0.1524" layer="91"/>
-<label x="149.86" y="35.56" size="1.778" layer="95"/>
-</segment>
-</net>
