File: HW6/TFTLCD/TFTLCD.sch (EAGLE design)
At the start: 22 parts, among them J1 USB-MB-H

Commit message: Progress on HW6
Parts:
- added U$10: TFTLCD, gen433:TFTLCD
Connections:
- net +3V3: now also U$10.1.LED, U$10.5.RESET, U$10.8.VCC
- net A1: now also U$10.3.SDA
- net B14: now also U$10.2.SCK
- net B15: now also U$10.4.A0
- net B7: now also U$10.6.CS
- net GND: now also U$10.7.GND
Changed lines of the file:
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@@
 <part name="P+3" library="433" deviceset="+5V" device=""/>
 <part name="+3V8" library="433" deviceset="+3V3" device=""/>
+<part name="U$10" library="gen433" deviceset="TFTLCD" device=""/>
+<part name="+3V9" library="gen433" deviceset="+3V3" device=""/>
+<part name="+3V10" library="gen433" deviceset="+3V3" device=""/>
+<part name="+3V11" library="gen433" deviceset="+3V3" device=""/>
+<part name="GND20" library="gen433" deviceset="GND" device=""/>
 </parts>
 <sheets>
@@
 <instance part="P+3" gate="1" x="236.22" y="121.92"/>
 <instance part="+3V8" gate="G$1" x="91.44" y="55.88"/>
+<instance part="U$10" gate="G$1" x="55.88" y="-27.94"/>
+<instance part="+3V9" gate="G$1" x="20.32" y="-12.7"/>
+<instance part="+3V10" gate="G$1" x="20.32" y="-43.18"/>
+<instance part="+3V11" gate="G$1" x="20.32" y="-66.04"/>
+<instance part="GND20" gate="1" x="20.32" y="-58.42" rot="R180"/>
 </instances>
 <busses>
@@
 <pinref part="GND10" gate="1" pin="GND"/>
 <wire x1="157.48" y1="27.94" x2="157.48" y2="33.02" width="0.1524" layer="91"/>
+</segment>
+<segment>
+<pinref part="U$10" gate="G$1" pin="7.GND"/>
+<pinref part="GND20" gate="1" pin="GND"/>
+<wire x1="38.1" y1="-60.96" x2="20.32" y2="-60.96" width="0.1524" layer="91"/>
 </segment>
 </net>
@@
 <wire x1="68.58" y1="53.34" x2="91.44" y2="53.34" width="0.1524" layer="91"/>
 </segment>
+<segment>
+<pinref part="U$10" gate="G$1" pin="8.VCC"/>
+<pinref part="+3V11" gate="G$1" pin="+3V3"/>
+<wire x1="38.1" y1="-68.58" x2="20.32" y2="-68.58" width="0.1524" layer="91"/>
+</segment>
+<segment>
+<pinref part="U$10" gate="G$1" pin="5.RESET"/>
+<pinref part="+3V10" gate="G$1" pin="+3V3"/>
+<wire x1="38.1" y1="-45.72" x2="20.32" y2="-45.72" width="0.1524" layer="91"/>
+</segment>
+<segment>
+<pinref part="U$10" gate="G$1" pin="1.LED"/>
+<wire x1="38.1" y1="-15.24" x2="20.32" y2="-15.24" width="0.1524" layer="91"/>
+<pinref part="+3V9" gate="G$1" pin="+3V3"/>
+</segment>
 </net>
 <net name="N$2" class="0">
@@
 <label x="187.96" y="132.08" size="1.778" layer="95" rot="MR0"/>
 </segment>
+<segment>
+<pinref part="U$10" gate="G$1" pin="3.SDA"/>
+<wire x1="38.1" y1="-30.48" x2="30.48" y2="-30.48" width="0.1524" layer="91"/>
+<label x="27.94" y="-30.48" size="1.778" layer="95"/>
+</segment>
 </net>
 <net name="PGD" class="0">
@@
 <label x="226.06" y="134.62" size="1.778" layer="95"/>
 </segment>
+<segment>
+<pinref part="U$10" gate="G$1" pin="4.A0"/>
+<wire x1="38.1" y1="-38.1" x2="30.48" y2="-38.1" width="0.1524" layer="91"/>
+<label x="27.94" y="-38.1" size="1.778" layer="95"/>
+</segment>
 </net>
 <net name="B14" class="0">
@@
 <label x="228.6" y="132.08" size="1.778" layer="95"/>
 </segment>
+<segment>
+<pinref part="U$10" gate="G$1" pin="2.SCK"/>
+<wire x1="38.1" y1="-22.86" x2="30.48" y2="-22.86" width="0.1524" layer="91"/>
+<label x="27.94" y="-22.86" size="1.778" layer="95"/>
+</segment>
 </net>
 <net name="B13" class="0">
@@
 <label x="226.06" y="121.92" size="1.778" layer="95"/>
 </segment>
-</net>
+<segment>
+<pinref part="U$10" gate="G$1" pin="6.CS"/>
+<wire x1="38.1" y1="-53.34" x2="30.48" y2="-53.34" width="0.1524" layer="91"/>
+<label x="27.94" y="-53.34" size="1.778" layer="95"/>
+</segment>
+</net>
